File: schematics/matrix-sq-v1.kicad_pcb (KiCad board)
At the start: 2 copper layers, 135 parts, among them J1 trg in 2, J2 trg in 1, J3 CV1, J4 CV2, J5 CV3, J6 Power, Q1 Q_NPN_BCE, Q2 Q_NPN_BCE, SW1 SW_Push, SW2 SW_Push, SW3 SW_Push, SW4 SW_Push, U1 TL084, X1 SW_Push, X2 SW_Push, X3 SW_Push, X4 SW_Push, X5 SW_Push, X6 SW_Push, Y1 SW_Push, Y2 SW_Push, Y3 SW_Push, Y4 SW_Push, Y5 SW_Push, Y6 SW_Push, Y7 Crystal

Commit message: front PCB
Parts:
- conFe1: value Conn_01x12_Female -> Conn_01x13_Female; footprint Connector_PinHeader_1.00mm:PinHeader_1x12_P1.00mm_Vertical -> Connector_PinHeader_1.00mm:PinHeader_1x13_P1.00mm_Vertical
- conFe2: value Conn_01x16_Female -> Conn_01x18_Female; footprint Connector_PinHeader_1.00mm:PinHeader_1x16_P1.00mm_Vertical -> Connector_PinHeader_1.00mm:PinHeader_1x18_P1.00mm_Vertical
- conMa1: value Conn_01x12_Male -> Conn_01x13_Male; footprint Connector_PinHeader_1.00mm:PinHeader_1x12_P1.00mm_Vertical -> Connector_PinHeader_1.00mm:PinHeader_1x13_P1.00mm_Vertical
- conMa2: value Conn_01x16_Male -> Conn_01x18_Male; footprint Connector_PinHeader_1.00mm:PinHeader_1x16_P1.00mm_Vertical -> Connector_PinHeader_1.00mm:PinHeader_1x18_P1.00mm_Vertical
- moved conMa2 334.8 mm to (145.0, 150.0), turned to 90 degrees
- moved conMa1 318.8 mm to (145.0, 221.5), turned to 90 degrees
- moved U1 222.4 mm to (176.8, 335.1), turned to 180 degrees
- moved R10 213.4 mm to (157.3, 321.5), turned to 180 degrees
- moved R9 205.1 mm to (164.5, 328.0), turned to -90 degrees
- moved fbc2 204.9 mm to (161.5, 330.2), turned to -90 degrees
- moved fbc1 193.4 mm to (161.5, 321.2), turned to 90 degrees
- moved R5 183.9 mm to (164.5, 324.3), turned to 90 degrees
- moved R7 173.7 mm to (161.5, 307.3), turned to 90 degrees
- moved R6 173.3 mm to (161.5, 295.8), turned to 90 degrees
- moved R8 171.4 mm to (160.8, 326.0), turned to 180 degrees
- moved J5 166.5 mm to (146.2, 314.0), turned to 90 degrees
- moved J4 153.3 mm to (146.2, 303.0), turned to 90 degrees
- moved J3 140.7 mm to (146.2, 292.0), turned to 90 degrees
- moved J1 125.7 mm to (146.2, 278.0), turned to 90 degrees
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- renumbered RV1 to A1, RV5 to A2, RV2 to A3, RV6 to A4, RV3 to A5, RV7 to A6, RV4 to A7, RV8 to A8, RV9 to B1, RV13 to B2, RV10 to B3, RV14 to B4, RV11 to B5, RV15 to B6, RV12 to B7, RV16 to B8, D2 to DLEDA2, D1 to LEDA1, D3 to LEDA3, D4 to LEDA4, D5 to LEDA5, D6 to LEDA6, D7 to LEDA7, D8 to LEDA8, D9 to LEDB1, D10 to LEDB2, D11 to LEDB3, D12 to LEDB4, D13 to LEDB5, D14 to LEDB6, D15 to LEDB7, D16 to LEDB8
Connections:
- net crystalA renamed crystalA-b
- net crystalB renamed crystalB-b
- net muxBit1 renamed muxBit1-b
- net muxBit2 renamed muxBit2-b
- net muxBit3 renamed muxBit3-b
- net muxReturnX renamed muxReturnX-b
- net muxReturnY renamed muxReturnY-b
- Atmega1 pad 14: Bit1 -> Bit1-b
- Atmega1 pad 15: Bit2 -> Bit2-b
- Atmega1 pad 16: Bit3 -> Bit3-b
- Atmega1 pad 17: load -> load-b
- Atmega1 pad 18: clk -> clk-b
- Atmega1 pad 19: din -> din-b
- Atmega1 pad 26: Bit4 -> Bit4-b
- Atmega1 pad 27: Bit5 -> Bit5-b
- Atmega1 pad 28: Bit6 -> Bit6-b
- Atmega1 pad 4: trig1 -> trig1ToAtmega-b
- Atmega1 pad 5: trig2 -> trig2ToAtmega-b
- J1 pad T: Net-(J1-PadT) -> trig2
- J2 pad T: Net-(J2-PadT) -> trig1
- Q1 pad 2: trig1 -> trg1ToAtmega-b
- Q2 pad 2: trig2 -> trg2ToAtmega-b
- conFe1 pad 1: +5V -> -12V
- conFe1 pad 10: Bit4 -> Bit3
- conFe1 pad 11: Bit5 -> Bit4
- conFe1 pad 12: Bit6 -> Bit5
- conFe1 pad 2: +12V -> +5V
- conFe1 pad 3: Earth -> +12V
- conFe1 pad 4: din -> Earth
- conFe1 pad 5: clk -> din
- conFe1 pad 6: load -> clk
- conFe1 pad 7: Bit1 -> load
- conFe1 pad 8: Bit2 -> Bit1
- conFe1 pad 9: Bit3 -> Bit2
- conFe2 pad 1: X1 -> trig1
- conFe2 pad 10: Y4 -> Y2
- conFe2 pad 11: Y5 -> Y3
- conFe2 pad 12: Y6 -> Y4
- conFe2 pad 13: menue1 -> Y5
- conFe2 pad 14: menue2 -> Y6
- conFe2 pad 15: menue3 -> menue1
- conFe2 pad 16: menue4 -> menue2
- conFe2 pad 2: X2 -> trig2
- conFe2 pad 3: X3 -> X6
- conFe2 pad 4: X4 -> X5
- conFe2 pad 5: X5 -> X4
- conFe2 pad 6: X6 -> X3
- conFe2 pad 7: Y1 -> X2
- conFe2 pad 8: Y2 -> X1
- conFe2 pad 9: Y3 -> Y1
- conMa1 pad 1: +5V -> -12V
- conMa1 pad 10: Bit4 -> Bit3-b
- conMa1 pad 11: Bit5 -> Bit4-b
- conMa1 pad 12: Bit6 -> Bit5-b
- conMa1 pad 2: +12V -> +5V
- conMa1 pad 3: Earth -> +12V
- conMa1 pad 4: din -> Earth
- conMa1 pad 5: clk -> din-b
- conMa1 pad 6: load -> clk-b
- conMa1 pad 7: Bit1 -> load-b
- conMa1 pad 8: Bit2 -> Bit1-b
- conMa1 pad 9: Bit3 -> Bit2-b
- conMa2 pad 1: X1 -> trig1-b
- conMa2 pad 10: Y4 -> Y2-b
- conMa2 pad 11: Y5 -> Y3-b
- conMa2 pad 12: Y6 -> Y4-b
- conMa2 pad 13: menue1 -> Y5-b
- conMa2 pad 14: menue2 -> Y6-b
- conMa2 pad 15: menue3 -> menue1-b
- conMa2 pad 16: menue4 -> menue2-b
- conMa2 pad 2: X2 -> trig2-b
- conMa2 pad 3: X3 -> X6-b
- conMa2 pad 4: X4 -> X5-b
- conMa2 pad 5: X5 -> X4-b
- conMa2 pad 6: X6 -> X3-b
- conMa2 pad 7: Y1 -> X2-b
- conMa2 pad 8: Y2 -> X1-b
- conMa2 pad 9: Y3 -> Y1-b
- dTrigIn1 pad 2: Net-(J2-PadT) -> trig2-b
- dTrigIn2 pad 2: Net-(J1-PadT) -> trig1-b
- muxX1 pad 1: X6 -> X6-b
- muxX1 pad 12: X5 -> X5-b
- muxX1 pad 13: X2 -> X2-b
- muxX1 pad 14: X3 -> X3-b
- muxX1 pad 15: X4 -> X4-b
- muxX1 pad 2: menue4 -> menue4-b
- muxX1 pad 4: X1 -> X1-b
- muxX1 pad 5: menue3 -> menue3-b
- muxY1 pad 1: Y6 -> Y6-b
- muxY1 pad 12: Y5 -> Y5-b
- muxY1 pad 13: Y2 -> Y2-b
- muxY1 pad 14: Y3 -> Y3-b
- muxY1 pad 15: Y4 -> Y4-b
- muxY1 pad 2: menue2 -> menue2-b
- muxY1 pad 4: Y1 -> Y1-b
- muxY1 pad 5: menue1 -> menue1-b
- trgRes1 pad 2: Net-(Q1-Pad1) -> Net-(Q2-Pad1)
- trgRes2 pad 2: Net-(Q2-Pad1) -> Net-(Q1-Pad1)
Routing:
- net +5V: track 0.00 -> 759.0 mm
- net Earth: track 0.00 -> 650.8 mm
- net clk: track 0.00 -> 195.4 mm
- net load: track 0.00 -> 189.6 mm
- net SQ1: track 0.00 -> 170.8 mm
- net Bit1: track 0.00 -> 170.6 mm
- net Bit2: track 0.00 -> 169.8 mm
- net Bit3: track 0.00 -> 169.8 mm
- net SQ2: track 0.00 -> 162.0 mm
- net din: track 0.00 -> 161.6 mm
- net Net-(R3-Pad2): track 0.00 -> 151.5 mm, vias 0 -> 1
- net Bit4: track 0.00 -> 145.3 mm
- net Bit5: track 0.00 -> 145.2 mm
- net Bit6: track 0.00 -> 145.0 mm
- net Pot B8: track 0.00 -> 140.4 mm
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
Commit message: pcb front and fill
Parts:
- SW1, SW2, SW3, SW4: moved to F.Cu
- moved C4 391.5 mm to (118.6, 149.4), turned to 90 degrees
- moved C8 386.2 mm to (123.4, 157.1), turned to 90 degrees
- moved C3 385.7 mm to (118.6, 157.1), turned to 90 degrees
- moved C2 379.1 mm to (116.2, 149.3), turned to 90 degrees
- moved C7 376.4 mm to (123.4, 146.6), turned to -90 degrees
- moved C1 373.2 mm to (116.2, 157.1), turned to 90 degrees
- moved C6 372.2 mm to (121.0, 149.4), turned to 90 degrees
- moved C5 364.9 mm to (121.0, 157.1), turned to 90 degrees
- moved voltageReg1 364.7 mm to (112.9, 165.3), turned to -90 degrees
- moved J6 310.9 mm to (110.5, 146.9)
- moved Y7 310.8 mm to (127.2, 207.9)
- moved C9 303.9 mm to (123.0, 204.7), turned to 90 degrees
- moved C10 294.5 mm to (131.4, 204.8), turned to 90 degrees
- moved Atmega1 291.1 mm to (170.0, 206.7), turned to -90 degrees
- moved muxX1 261.3 mm to (149.3, 182.0), turned to -90 degrees
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Connections:
- Atmega1 pad 4: trig1ToAtmega-b -> trg1ToAtmega-b
- Atmega1 pad 5: trig2ToAtmega-b -> trg2ToAtmega-b
Routing:
- net Earth: track 650.8 -> 902.4 mm
- net +5V: track 759.0 -> 993.5 mm
- net -12V: track 45.8 -> 180.3 mm
- net +12V: track 58.3 -> 177.8 mm
- net Y1-b: track 0.00 -> 84.1 mm, vias 0 -> 1
- net trg2ToAtmega-b: track 0.00 -> 76.3 mm
- net trg1ToAtmega-b: track 0.00 -> 70.3 mm
- net Y2-b: track 0.00 -> 68.9 mm
- net Y5-b: track 0.00 -> 68.2 mm
- net X5-b: track 0.00 -> 67.9 mm
- net Y3-b: track 0.00 -> 65.5 mm
- net X2-b: track 0.00 -> 64.0 mm
- net Y4-b: track 0.00 -> 59.6 mm
- net menue1-b: track 0.00 -> 59.3 mm
- net X4-b: track 0.00 -> 55.5 mm
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- added copper zone on B.Cu, net (none)
- added copper zone on F.Cu, net (none)
