File: schematics/matrix-sq-v1.kicad_pcb (KiCad board)
At the start: 2 copper layers, 135 parts, among them J1 trg in 2, J2 trg in 1, J3 CV1, J4 CV2, J5 CV3, J6 Power, Q1 Q_NPN_BCE, Q2 Q_NPN_BCE, SW1 SW_Push, SW2 SW_Push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

Commit message: refactor front-gerber
Parts:
- moved C7 14.5 mm to (129.8, 159.6), turned to 90 degrees
- moved C8 11.4 mm to (129.8, 147.6)
- moved C5 6.22 mm to (126.7, 159.6)
- moved C6 5.80 mm to (126.5, 147.6)
- moved C3 5.32 mm to (123.3, 159.6)
- moved C4 4.96 mm to (123.2, 147.6)
- moved C1 4.63 mm to (120.1, 159.6)
- moved C2 4.23 mm to (120.1, 147.7)
Routing:
- net Earth: track 902.4 -> 938.8 mm
- net +12V: track 177.8 -> 195.6 mm
- net -12V: track 180.3 -> 197.8 mm
Other:
- board text added: "Matrix - SQ with by Christian Grothe"

Commit message: edge cuts
Other:
- board outline added: 220.5 x 199.4 mm
Changed lines of the file:
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@@
   (gr_circle (center 109.95 204.83) (end 110.55 204.83) (layer "F.SilkS") (width 0.1) (fill solid))
   (gr_circle (center 109.97 205.64) (end 110.57 205.64) (layer "F.SilkS") (width 0.1) (fill solid))
+  (gr_rect (start 108.3 140.6) (end 182.7 227.7) (layer "Edge.Cuts") (width 0.1) (fill none))
+  (gr_rect (start 67 240) (end 287.5 340) (layer "Edge.Cuts") (width 0.1) (fill none))
   (gr_text "Matrix - SQ with   by Christian Grothe" (at 110.16 203.9 90) (layer "F.SilkS")
     (effects (font (size 1.5 1.5) (thickness 0.3)))

Commit message: new header footprints
Parts:
- added R?: 47k, Resistor_THT:R_Axial_DIN0207_L6.3mm_D2.5mm_P7.62mm_Horizontal, F.Cu at (275.9, 277.1)
- conFe1, conMa1: footprint Connector_PinHeader_1.00mm:PinHeader_1x13_P1.00mm_Vertical -> Connector_PinHeader_2.54mm:PinHeader_1x13_P2.54mm_Vertical
- conFe2: footprint Connector_PinHeader_1.00mm:PinHeader_1x18_P1.00mm_Vertical -> Connector_PinHeader_2.54mm:PinHeader_1x18_P2.54mm_Vertical
- conMa2: footprint Connector_PinHeader_1.00mm:PinHeader_1x18_P1.00mm_Vertical -> Connector_PinSocket_2.54mm:PinSocket_1x18_P2.54mm_Vertical
- moved U1 16.8 mm to (181.5, 319.0), turned to -90 degrees
- moved R9 9.89 mm to (154.8, 330.0), turned to 180 degrees
- moved fbc1 9.39 mm to (157.3, 329.6)
- moved conMa2 7.10 mm to (162.0, 135.5)
- moved conFe1 7.00 mm to (145.0, 337.0)
- moved R5 6.80 mm to (160.5, 329.8)
- moved fbc2 6.61 mm to (157.3, 325.1), turned to 90 degrees
- moved R8 6.20 mm to (154.6, 326.1)
- moved C8 3.60 mm to (129.7, 151.2)
- moved C2 3.60 mm to (120.0, 151.2)
- moved C4 3.60 mm to (123.1, 151.2)
- moved C6 3.60 mm to (126.4, 151.2)
- moved R10 3.01 mm to (154.5, 322.6)
Connections:
- Max1 pad 18: +5V -> Net-(Max1-Pad18)
Routing:
- net Net-(R8-Pad1): track 15.0 -> 67.4 mm, vias 0 -> 1
- net Net-(R3-Pad2): track 151.5 -> 201.3 mm, vias 1 -> 0
- net menue4-b: track 40.1 -> 71.8 mm
- net +12V: track 195.6 -> 167.9 mm
- net Net-(R10-Pad1): track 22.1 -> 47.5 mm
- net Net-(Max1-Pad18): track 0.00 -> 22.7 mm
- net Earth: track 938.8 -> 917.0 mm
- net Bit6-b: track 28.0 -> 47.8 mm
- net Bit5-b: track 25.1 -> 43.4 mm
- net Y6: track 119.6 -> 101.6 mm
- net menue2-b: track 49.1 -> 66.4 mm
- net Bit4-b: track 22.3 -> 39.1 mm
- net load: track 189.6 -> 172.8 mm
- net Y5: track 107.3 -> 90.9 mm
- net menue1-b: track 59.3 -> 75.4 mm
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Other:
- board size 220.5 x 199.4 mm -> 220.5 x 208.8 mm
