File: schematics/matrix-sq-v1.kicad_pcb (KiCad board)
At the start: 2 copper layers, 220.5 x 208.8 mm, 136 parts, among them J1 trg in 2, J2 trg in 1, J3 CV1, J4 CV2, J5 CV3, J6 Power, Q1 Q_NPN_BCE, Q2 Q_NPN_BCE, SW1 SW_Push, SW2 SW_Push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

Commit message: refactor 6.8.
Parts:
- added J?: Conn_01x02_Female, Connector_PinHeader_2.54mm:PinHeader_1x02_P2.54mm_Vertical, F.Cu at (174.0, 212.8)
- added R12: R600, Resistor_THT:R_Axial_DIN0207_L6.3mm_D2.5mm_P7.62mm_Horizontal, F.Cu at (166.3, 187.3)
- added R13: 10k, Resistor_THT:R_Axial_DIN0207_L6.3mm_D2.5mm_P7.62mm_Horizontal, F.Cu at (166.4, 182.9)
- added R14: 10k, Resistor_THT:R_Axial_DIN0207_L6.3mm_D2.5mm_P7.62mm_Horizontal, F.Cu at (166.4, 178.5)
- added R15: 10k, Resistor_THT:R_Axial_DIN0207_L6.3mm_D2.5mm_P7.62mm_Horizontal, F.Cu at (166.3, 191.7)
- added R16: 10k, Resistor_THT:R_Axial_DIN0207_L6.3mm_D2.5mm_P7.62mm_Horizontal, F.Cu at (166.5, 169.6)
- added R17: 10k, Resistor_THT:R_Axial_DIN0207_L6.3mm_D2.5mm_P7.62mm_Horizontal, F.Cu at (166.3, 200.8)
- added R18: 10k, Resistor_THT:R_Axial_DIN0207_L6.3mm_D2.5mm_P7.62mm_Horizontal, F.Cu at (166.5, 174.1)
- added R19: 10k, Resistor_THT:R_Axial_DIN0207_L6.3mm_D2.5mm_P7.62mm_Horizontal, F.Cu at (166.3, 196.3)
- added R20: 10k, Resistor_THT:R_Axial_DIN0207_L6.3mm_D2.5mm_P7.62mm_Horizontal, F.Cu at (127.7, 199.4)
- added R21: 10k, Resistor_THT:R_Axial_DIN0207_L6.3mm_D2.5mm_P7.62mm_Horizontal, F.Cu at (127.7, 191.0)
- added R22: 10k, Resistor_THT:R_Axial_DIN0207_L6.3mm_D2.5mm_P7.62mm_Horizontal, F.Cu at (127.7, 182.5)
- added R23: 10k, Resistor_THT:R_Axial_DIN0207_L6.3mm_D2.5mm_P7.62mm_Horizontal, F.Cu at (127.7, 203.6)
- added R24: 10k, Resistor_THT:R_Axial_DIN0207_L6.3mm_D2.5mm_P7.62mm_Horizontal, F.Cu at (127.6, 173.6)
- added R25: 10k, Resistor_THT:R_Axial_DIN0207_L6.3mm_D2.5mm_P7.62mm_Horizontal, F.Cu at (127.7, 195.2)
- added R26: 10k, Resistor_THT:R_Axial_DIN0207_L6.3mm_D2.5mm_P7.62mm_Horizontal, F.Cu at (127.7, 177.9)
- added R27: 10k, Resistor_THT:R_Axial_DIN0207_L6.3mm_D2.5mm_P7.62mm_Horizontal, F.Cu at (127.7, 186.8)
- moved Max1 68.3 mm to (220.3, 337.3), turned to 90 degrees
- moved R? 63.9 mm to (254.3, 337.2), turned to 90 degrees
- moved muxY1 20.9 mm to (152.3, 179.1), turned to 0 degrees
- moved muxX1 11.7 mm to (138.0, 179.1), turned to 0 degrees
- moved Q1 11.1 mm to (170.5, 154.2)
- moved Q2 11.1 mm to (154.1, 154.2)
- moved trigin2 11.1 mm to (160.6, 161.6)
- moved trigin1 11.1 mm to (164.8, 161.6)
- moved dTrigIn1 11.0 mm to (153.1, 150.5)
- moved trgRes2 11.0 mm to (171.7, 149.0)
- moved trgRes1 11.0 mm to (159.3, 149.0)
- moved dTrigIn2 11.0 mm to (165.3, 150.7)
- moved Y7 7.58 mm to (124.0, 214.8), turned to 0 degrees
- moved C9 4.84 mm to (124.3, 209.3), turned to 180 degrees
- moved C10 4.73 mm to (129.8, 209.3), turned to 180 degrees
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Connections:
- Atmega1 pad 2: unconnected-(Atmega1-Pad2) -> RX
- Atmega1 pad 3: unconnected-(Atmega1-Pad3) -> TX
Routing:
- net Bit3: track 181.7 -> 96.0 mm
- net load: track 172.8 -> 92.2 mm
- net clk: track 180.2 -> 102.0 mm
- net din: track 147.9 -> 69.7 mm
- net Column3: track 155.7 -> 77.7 mm
- net Column1: track 166.6 -> 90.8 mm
- net Column2: track 183.3 -> 108.6 mm
- net Column5: track 170.1 -> 99.1 mm
- net Column4: track 145.2 -> 77.2 mm
- net Row1: track 102.2 -> 162.1 mm
- net X6-b: track 54.1 -> 105.5 mm
- net X1-b: track 47.6 -> 96.6 mm
- net Row6: track 120.8 -> 74.9 mm
- net Column6: track 124.0 -> 90.0 mm
- net menue3-b: track 55.6 -> 87.8 mm
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- added copper zone on B.Cu, net Earth
- removed copper zone on B.Cu, net (none)
- removed copper zone on F.Cu, net (none)
Other:
- board size 220.5 x 208.8 mm -> 200 x 208.1 mm
- board text added: "10k"

Commit message: refactor
Parts:
- J: renamed from J?; value Conn_01x02_Female -> Conn_01x03_Female; footprint Connector_PinHeader_2.54mm:PinHeader_1x02_P2.54mm_Vertical -> Connector_PinHeader_2.54mm:PinHeader_1x03_P2.54mm_Vertical
Connections:
- Atmega1 pad 1: unconnected-(Atmega1-Pad1) -> RESET
- J pad 1: RX -> RESET
- J pad 2: TX -> RX
- U1 pad 11: -12V -> (no net)
- U1 pad 4: +12V -> (no net)
Routing:
- net Row2: track 70.7 -> 127.2 mm
- net RESET: track 0.00 -> 6.18 mm
- net TX: track 12.3 -> 13.4 mm
Other:
- board text added: ".1u"
- board text added: "1,5k"
- board text added: "10u"
- board text added: "200k"
- board text added: "22pf"
- board text added: "47k"
- board text added: "RX"
- board text added: "TX"
- board text added: "res"
