File: schematics/matrix-sq-v1.kicad_sch (KiCad schematic)
At the start: 135 parts, among them J1 trg in 2, J2 trg in 1, J3 CV1, J4 CV2, J5 CV3, J6 Power, Q1 Q_NPN_BCE, Q2 Q_NPN_BCE, SW1 SW_Push, SW2 SW_Push, SW3 SW_Push, SW4 SW_Push, U1 TL084, X1 SW_Push, X2 SW_Push, X3 SW_Push, X4 SW_Push, X5 SW_Push, X6 SW_Push, Y1 SW_Push, Y2 SW_Push, Y3 SW_Push, Y4 SW_Push, Y5 SW_Push, Y6 SW_Push, Y7 Crystal

Commit message: front PCB
Parts:
- conFe1: value Conn_01x12_Female -> Conn_01x13_Female; footprint Connector_PinHeader_1.00mm:PinHeader_1x12_P1.00mm_Vertical -> Connector_PinHeader_1.00mm:PinHeader_1x13_P1.00mm_Vertical; symbol Connector:Conn_01x12_Female -> Connector:Conn_01x13_Female
- conFe2: value Conn_01x16_Female -> Conn_01x18_Female; footprint Connector_PinHeader_1.00mm:PinHeader_1x16_P1.00mm_Vertical -> Connector_PinHeader_1.00mm:PinHeader_1x18_P1.00mm_Vertical; symbol Connector:Conn_01x16_Female -> Connector:Conn_01x18_Female
- conMa1: value Conn_01x12_Male -> Conn_01x13_Male; footprint Connector_PinHeader_1.00mm:PinHeader_1x12_P1.00mm_Vertical -> Connector_PinHeader_1.00mm:PinHeader_1x13_P1.00mm_Vertical; symbol Connector:Conn_01x12_Male -> Connector:Conn_01x13_Male
- conMa2: value Conn_01x16_Male -> Conn_01x18_Male; footprint Connector_PinHeader_1.00mm:PinHeader_1x16_P1.00mm_Vertical -> Connector_PinHeader_1.00mm:PinHeader_1x18_P1.00mm_Vertical; symbol Connector:Conn_01x16_Male -> Connector:Conn_01x18_Male
- renumbered RV1 to A1, RV5 to A2, RV2 to A3, RV6 to A4, RV3 to A5, RV7 to A6, RV4 to A7, RV8 to A8, RV9 to B1, RV13 to B2, RV10 to B3, RV14 to B4, RV11 to B5, RV15 to B6, RV12 to B7, RV16 to B8, D2 to DLEDA2, D1 to LEDA1, D3 to LEDA3, D4 to LEDA4, D5 to LEDA5, D6 to LEDA6, D7 to LEDA7, D8 to LEDA8, D9 to LEDB1, D10 to LEDB2, D11 to LEDB3, D12 to LEDB4, D13 to LEDB5, D14 to LEDB6, D15 to LEDB7, D16 to LEDB8
Connections:
- net +12V: now also conFe1.3 (Pin_3), conMa1.3 (Pin_3); no longer conFe1.2 (Pin_2), conMa1.2 (Pin_2)
- net +5V: now also conFe1.2 (Pin_2), conMa1.2 (Pin_2); no longer conFe1.1 (Pin_1), conMa1.1 (Pin_1)
- net -12V: now also conFe1.1 (Pin_1), conMa1.1 (Pin_1)
- net Bit1: now also conFe1.8 (Pin_8); no longer Atmega1.14 (PB0), conFe1.7 (Pin_7), conMa1.7 (Pin_7)
- net Bit2: now also conFe1.9 (Pin_9); no longer Atmega1.15 (PB1), conFe1.8 (Pin_8), conMa1.8 (Pin_8)
- net Bit3: now also conFe1.10 (Pin_10); no longer Atmega1.16 (PB2), conFe1.9 (Pin_9), conMa1.9 (Pin_9)
- net Bit4: now also conFe1.11 (Pin_11); no longer Atmega1.26 (PC3), conFe1.10 (Pin_10), conMa1.10 (Pin_10)
- net Bit5: now also conFe1.12 (Pin_12); no longer Atmega1.27 (PC4), conFe1.11 (Pin_11), conMa1.11 (Pin_11)
- net Bit6: now also conFe1.13 (Pin_13); no longer Atmega1.28 (PC5), conFe1.12 (Pin_12), conMa1.12 (Pin_12)
- net Earth: now also conFe1.4 (Pin_4), conMa1.4 (Pin_4); no longer conFe1.3 (Pin_3), conMa1.3 (Pin_3)
- net X1: now also conFe2.8 (Pin_8); no longer conFe2.1 (Pin_1), conMa2.1 (Pin_1), muxX1.4 (A7)
- net X2: now also conFe2.7 (Pin_7); no longer conFe2.2 (Pin_2), conMa2.2 (Pin_2), muxX1.13 (A0)
- net X3: now also conFe2.6 (Pin_6); no longer conFe2.3 (Pin_3), conMa2.3 (Pin_3), muxX1.14 (A1)
- net X4: now also conFe2.5 (Pin_5); no longer conFe2.4 (Pin_4), conMa2.4 (Pin_4), muxX1.15 (A2)
- net X5: now also conFe2.4 (Pin_4); no longer conFe2.5 (Pin_5), conMa2.5 (Pin_5), muxX1.12 (A3)
- net X6: now also conFe2.3 (Pin_3); no longer conFe2.6 (Pin_6), conMa2.6 (Pin_6), muxX1.1 (A4)
- net Y1: now also conFe2.9 (Pin_9); no longer conFe2.7 (Pin_7), conMa2.7 (Pin_7), muxY1.4 (A7)
- net Y2: now also conFe2.10 (Pin_10); no longer conFe2.8 (Pin_8), conMa2.8 (Pin_8), muxY1.13 (A0)
- net Y3: now also conFe2.11 (Pin_11); no longer conFe2.9 (Pin_9), conMa2.9 (Pin_9), muxY1.14 (A1)
- net Y4: now also conFe2.12 (Pin_12); no longer conFe2.10 (Pin_10), conMa2.10 (Pin_10), muxY1.15 (A2)
- net Y5: now also conFe2.13 (Pin_13); no longer conFe2.11 (Pin_11), conMa2.11 (Pin_11), muxY1.12 (A3)
- net Y6: now also conFe2.14 (Pin_14); no longer conFe2.12 (Pin_12), conMa2.12 (Pin_12), muxY1.1 (A4)
- net clk: now also conFe1.6 (Pin_6); no longer Atmega1.18 (PB4), conFe1.5 (Pin_5), conMa1.5 (Pin_5)
- net din: now also conFe1.5 (Pin_5); no longer Atmega1.19 (PB5), conFe1.4 (Pin_4), conMa1.4 (Pin_4)
- net load: now also conFe1.7 (Pin_7); no longer Atmega1.17 (PB3), conFe1.6 (Pin_6), conMa1.6 (Pin_6)
- net menue1: now also conFe2.15 (Pin_15); no longer conFe2.13 (Pin_13), conMa2.13 (Pin_13), muxY1.5 (A5)
- net menue2: now also conFe2.16 (Pin_16); no longer conFe2.14 (Pin_14), conMa2.14 (Pin_14), muxY1.2 (A6)
- net menue3: now also conFe2.17 (Pin_17); no longer conFe2.15 (Pin_15), conMa2.15 (Pin_15), muxX1.5 (A5)
- net menue4: now also conFe2.18 (Pin_18); no longer conFe2.16 (Pin_16), conMa2.16 (Pin_16), muxX1.2 (A6)
- net trig1: now also J2.T, conFe2.1 (Pin_1); no longer Atmega1.4 (PD2), Q1.2 (C)
- net trig2: now also J1.T, conFe2.2 (Pin_2); no longer Atmega1.5 (PD3), Q2.2 (C)
- net at trgRes1.2: now also Q2.1 (B); no longer Q1.1 (B)
- net trig2-b: now reaches dTrigIn1.2 (A)
- net trig2-b: now also conMa2.2 (Pin_2); no longer J2.T
- net trig1-b: now reaches dTrigIn2.2 (A)
- net trig1-b: now also conMa2.1 (Pin_1); no longer J1.T
- net at trgRes2.2: now also Q1.1 (B); no longer Q2.1 (B)
- net crystalA renamed crystalA-b
- net crystalB renamed crystalB-b
- net muxBit1 renamed muxBit1-b
- net muxBit2 renamed muxBit2-b
- net muxBit3 renamed muxBit3-b
- net muxReturnX renamed muxReturnX-b
- net muxReturnY renamed muxReturnY-b
- new net Bit1-b: Atmega1.14 (PB0), conMa1.8 (Pin_8)
- new net Bit2-b: Atmega1.15 (PB1), conMa1.9 (Pin_9)
- new net Bit3-b: Atmega1.16 (PB2), conMa1.10 (Pin_10)
- new net Bit4-b: Atmega1.26 (PC3), conMa1.11 (Pin_11)
- new net Bit5-b: Atmega1.27 (PC4), conMa1.12 (Pin_12)
- new net Bit6-b: Atmega1.28 (PC5), conMa1.13 (Pin_13)
- new net X1-b: conMa2.8 (Pin_8), muxX1.4 (A7)
- new net X2-b: conMa2.7 (Pin_7), muxX1.13 (A0)
- new net X3-b: conMa2.6 (Pin_6), muxX1.14 (A1)
- new net X4-b: conMa2.5 (Pin_5), muxX1.15 (A2)
- new net X5-b: conMa2.4 (Pin_4), muxX1.12 (A3)
- new net X6-b: conMa2.3 (Pin_3), muxX1.1 (A4)
- new net Y1-b: conMa2.9 (Pin_9), muxY1.4 (A7)
- new net Y2-b: conMa2.10 (Pin_10), muxY1.13 (A0)
- new net Y3-b: conMa2.11 (Pin_11), muxY1.14 (A1)
- new net Y4-b: conMa2.12 (Pin_12), muxY1.15 (A2)
- new net Y5-b: conMa2.13 (Pin_13), muxY1.12 (A3)
- new net Y6-b: conMa2.14 (Pin_14), muxY1.1 (A4)
- new net clk-b: Atmega1.18 (PB4), conMa1.6 (Pin_6)
- new net din-b: Atmega1.19 (PB5), conMa1.5 (Pin_5)
- new net load-b: Atmega1.17 (PB3), conMa1.7 (Pin_7)
- new net menue1-b: conMa2.15 (Pin_15), muxY1.5 (A5)
- new net menue2-b: conMa2.16 (Pin_16), muxY1.2 (A6)
- new net menue3-b: conMa2.17 (Pin_17), muxX1.5 (A5)
- new net menue4-b: conMa2.18 (Pin_18), muxX1.2 (A6)
- new net trg1ToAtmega-b: Q1.2 (C)
- new net trg2ToAtmega-b: Q2.2 (C)
- new net trig1ToAtmega-b: Atmega1.4 (PD2)
- new net trig2ToAtmega-b: Atmega1.5 (PD3)

Commit message: pcb front and fill
Connections:
- net trig1ToAtmega-b is gone; now on net trg1ToAtmega-b: Atmega1.4 (PD2)
- net trig2ToAtmega-b is gone; now on net trg2ToAtmega-b: Atmega1.5 (PD3)

Commit message: new header footprints
Parts:
- added R11: 47k, Resistor_THT:R_Axial_DIN0207_L6.3mm_D2.5mm_P7.62mm_Horizontal, symbol Device:R
- conFe1, conMa1: footprint Connector_PinHeader_1.00mm:PinHeader_1x13_P1.00mm_Vertical -> Connector_PinHeader_2.54mm:PinHeader_1x13_P2.54mm_Vertical
- conFe2: footprint Connector_PinHeader_1.00mm:PinHeader_1x18_P1.00mm_Vertical -> Connector_PinHeader_2.54mm:PinHeader_1x18_P2.54mm_Vertical
- conMa2: footprint Connector_PinHeader_1.00mm:PinHeader_1x18_P1.00mm_Vertical -> Connector_PinSocket_2.54mm:PinSocket_1x18_P2.54mm_Vertical
Connections:
- net +5V: now also R11.1; no longer Max1.18 (ISET)
- new net: Max1.18 (ISET), R11.2
Changed lines of the file:
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@@
   (junction (at 452.12 256.54) (diameter 0) (color 0 0 0 0)
   )
-  (junction (at 176.53 326.39) (diameter 0) (color 0 0 0 0)
-  )
   (junction (at 408.94 45.72) (diameter 0) (color 0 0 0 0)
   )
@@
       (effects (font (size 1.27 1.27)) (justify left))
     )
-    (property "Footprint" "Connector_PinHeader_1.00mm:PinHeader_1x18_P1.00mm_Vertical" (id 2) (at 284.48 260.35 0)
+    (property "Footprint" "Connector_PinHeader_2.54mm:PinHeader_1x18_P2.54mm_Vertical" (id 2) (at 284.48 260.35 0)
       (effects (font (size 1.27 1.27)) hide)
     )
@@
     (property "Reference" "conMa2" (id 0) (at 541.655 67.31 0))
     (property "Value" "Conn_01x18_Male" (id 1) (at 541.655 69.85 0))
-    (property "Footprint" "Connector_PinHeader_1.00mm:PinHeader_1x18_P1.00mm_Vertical" (id 2) (at 541.02 90.17 0)
+    (property "Footprint" "Connector_PinSocket_2.54mm:PinSocket_1x18_P2.54mm_Vertical" (id 2) (at 541.02 90.17 0)
       (effects (font (size 1.27 1.27)) hide)
     )
@@
       (effects (font (size 1.27 1.27)) (justify left))
     )
-    (property "Footprint" "Connector_PinHeader_1.00mm:PinHeader_1x13_P1.00mm_Vertical" (id 2) (at 260.35 255.27 0)
+    (property "Footprint" "Connector_PinHeader_2.54mm:PinHeader_1x13_P2.54mm_Vertical" (id 2) (at 260.35 255.27 0)
       (effects (font (size 1.27 1.27)) hide)
     )
@@
     (pin "1")
   )
+  (symbol (lib_id "Device:R") (at 172.72 326.39 90) (unit 1)
+    (in_bom yes) (on_board yes) (fields_autoplaced)
+    (property "Reference" "R11" (id 0) (at 172.72 320.04 90))
+    (property "Value" "47k" (id 1) (at 172.72 322.58 90))
+    (property "Footprint" "Resistor_THT:R_Axial_DIN0207_L6.3mm_D2.5mm_P7.62mm_Horizontal" (id 2) (at 172.72 328.168 90)
+      (effects (font (size 1.27 1.27)) hide)
+    )
+    (property "Datasheet" "~" (id 3) (at 172.72 326.39 0)
+      (effects (font (size 1.27 1.27)) hide)
+    )
+    (property "Datasheet" "~" (id 4) (at 172.72 326.39 0)
+      (effects (font (size 1.27 1.27)) hide)
+    )
+    (property "Reference" "R?" (id 5) (at 172.72 326.39 0)
+      (effects (font (size 1.27 1.27)) hide)
+    )
+    (property "Value" "47k" (id 6) (at 172.72 326.39 0)
+      (effects (font (size 1.27 1.27)) hide)
+    )
+    (pin "1")
+    (pin "2")
+  )
   (symbol (lib_id "power:Earth") (at 139.7 34.29 0) (unit 1)
     (in_bom yes) (on_board yes) (fields_autoplaced)
@@
     (pin "1")
   )
-  (symbol (lib_id "power:+5V") (at 176.53 326.39 90) (unit 1)
-    (in_bom yes) (on_board yes) (fields_autoplaced)
-    (property "Reference" "#PWR0181" (id 0) (at 180.34 326.39 0)
+  (symbol (lib_id "power:+5V") (at 168.91 326.39 90) (unit 1)
+    (in_bom yes) (on_board yes)
+    (property "Reference" "#PWR0181" (id 0) (at 172.72 326.39 0)
       (effects (font (size 1.27 1.27)) hide)
     )
-    (property "Value" "+5V" (id 1) (at 172.72 326.3899 90)
+    (property "Value" "+5V" (id 1) (at 168.91 323.85 90)
       (effects (font (size 1.27 1.27)) (justify left))
     )
-    (property "Footprint" "" (id 2) (at 176.53 326.39 0)
+    (property "Footprint" "" (id 2) (at 168.91 326.39 0)
       (effects (font (size 1.27 1.27)) hide)
     )
-    (property "Datasheet" "" (id 3) (at 176.53 326.39 0)
+    (property "Datasheet" "" (id 3) (at 168.91 326.39 0)
       (effects (font (size 1.27 1.27)) hide)
     )
@@
     (property "Reference" "conMa1" (id 0) (at 509.27 63.5 0))
     (property "Value" "Conn_01x13_Male" (id 1) (at 509.27 66.04 0))
-    (property "Footprint" "Connector_PinHeader_1.00mm:PinHeader_1x13_P1.00mm_Vertical" (id 2) (at 509.27 85.09 0)
+    (property "Footprint" "Connector_PinHeader_2.54mm:PinHeader_1x13_P2.54mm_Vertical" (id 2) (at 509.27 85.09 0)
       (effects (font (size 1.27 1.27)) hide)
     )
@@
     (pin "2")
   )
-  (symbol (lib_id "power:+5V") (at 176.53 326.39 90) (unit 1)
-    (in_bom yes) (on_board yes) (fields_autoplaced)
-    (property "Reference" "#PWR0180" (id 0) (at 180.34 326.39 0)
-      (effects (font (size 1.27 1.27)) hide)
-    )
-    (property "Value" "+5V" (id 1) (at 172.72 326.3899 90)
-      (effects (font (size 1.27 1.27)) (justify left))
-    )
-    (property "Footprint" "" (id 2) (at 176.53 326.39 0)
-      (effects (font (size 1.27 1.27)) hide)
-    )
-    (property "Datasheet" "" (id 3) (at 176.53 326.39 0)
-      (effects (font (size 1.27 1.27)) hide)
-    )
-    (pin "1")
-  )
   (symbol (lib_id "power:Earth") (at 105.41 31.75 180) (unit 1)
     (in_bom yes) (on_board yes) (fields_autoplaced)
@@
       (reference "#PWR0179") (unit 1) (value "+5V") (footprint "")
     )
-    (path "/e4ad1db8-77ee-40e1-a2ab-691ed735e151"
-      (reference "#PWR0180") (unit 1) (value "+5V") (footprint "")
-    )
     (path "/b9fb5a36-0af2-4b8d-b921-087e1d790a72"
       (reference "#PWR0181") (unit 1) (value "+5V") (footprint "")
@@
       (reference "R10") (unit 1) (value "1,5k") (footprint "Resistor_THT:R_Axial_DIN0207_L6.3mm_D2.5mm_P7.62mm_Horizontal")
     )
+    (path "/83eaba9f-77d3-4299-9449-d2247fd790dc"
+      (reference "R11") (unit 1) (value "47k") (footprint "Resistor_THT:R_Axial_DIN0207_L6.3mm_D2.5mm_P7.62mm_Horizontal")
+    )
     (path "/6c3df62d-46ed-4378-9a4c-b3145d0eaec9"
       (reference "SQ1Led1") (unit 1) (value "74HC4051") (footprint "Package_DIP:DIP-16_W7.62mm_Socket")
@@
     )
     (path "/74d2e6c1-2ca5-480e-9500-ae355181aedc"
-      (reference "conFe1") (unit 1) (value "Conn_01x13_Female") (footprint "Connector_PinHeader_1.00mm:PinHeader_1x13_P1.00mm_Vertical")
+      (reference "conFe1") (unit 1) (value "Conn_01x13_Female") (footprint "Connector_PinHeader_2.54mm:PinHeader_1x13_P2.54mm_Vertical")
     )
     (path "/00d51d94-c5b2-416a-9abe-6b7e1e4602f3"
-      (reference "conFe2") (unit 1) (value "Conn_01x18_Female") (footprint "Connector_PinHeader_1.00mm:PinHeader_1x18_P1.00mm_Vertical")
+      (reference "conFe2") (unit 1) (value "Conn_01x18_Female") (footprint "Connector_PinHeader_2.54mm:PinHeader_1x18_P2.54mm_Vertical")
     )
     (path "/c5f0fbd0-afb8-4f71-9e50-9a86356072e6"
-      (reference "conMa1") (unit 1) (value "Conn_01x13_Male") (footprint "Connector_PinHeader_1.00mm:PinHeader_1x13_P1.00mm_Vertical")
+      (reference "conMa1") (unit 1) (value "Conn_01x13_Male") (footprint "Connector_PinHeader_2.54mm:PinHeader_1x13_P2.54mm_Vertical")
     )
     (path "/43fe4313-e2a7-479b-8151-e8cce48d9fa7"
-      (reference "conMa2") (unit 1) (value "Conn_01x18_Male") (footprint "Connector_PinHeader_1.00mm:PinHeader_1x18_P1.00mm_Vertical")
+      (reference "conMa2") (unit 1) (value "Conn_01x18_Male") (footprint "Connector_PinSocket_2.54mm:PinSocket_1x18_P2.54mm_Vertical")
     )
     (path "/1f68fad2-b1d9-4f0c-abc3-91d54f436fdb"

Commit message: refactor 6.8.
Parts:
- added J7: Conn_01x02_Female, Connector_PinHeader_2.54mm:PinHeader_1x02_P2.54mm_Vertical, symbol Connector:Conn_01x02_Female
- added R12: R600, Resistor_THT:R_Axial_DIN0207_L6.3mm_D2.5mm_P7.62mm_Horizontal, symbol Device:R
- added R13, R14, R15, R16, R17, R18, R19, R20, R21, R22, R23, R24, R25, R26, R27: 10k, Resistor_THT:R_Axial_DIN0207_L6.3mm_D2.5mm_P7.62mm_Horizontal, symbol Device:R
Connections:
- net Earth: now also R12.2, R13.2, R14.2, R15.2, R16.2, R17.2, R18.2, R19.2, R20.2, R21.2, R22.2, R23.2, R24.2, R25.2, R26.2, R27.2
- net X1-b: now also R27.1
- net X2-b: now also R20.1
- net X3-b: now also R21.1
- net X4-b: now also R22.1
- net X5-b: now also R23.1
- net X6-b: now also R24.1
- net Y1-b: now also R19.1
- net Y2-b: now also R12.1
- net Y3-b: now also R13.1
- net Y4-b: now also R14.1
- net Y5-b: now also R15.1
- net Y6-b: now also R16.1
- net menue1-b: now also R17.1
- net menue2-b: now also R18.1
- net menue3-b: now also R25.1
- net menue4-b: now also R26.1
- net RX: now reaches Atmega1.2 (PD0)
- net RX: now also J7.1 (Pin_1)
- net TX: now reaches Atmega1.3 (PD1)
- net TX: now also J7.2 (Pin_2)
- no-connect marks 11 -> 9
Other:
- moved on the sheet: muxX1, muxY1

Commit message: refactor
Parts:
- J: renamed from J7; value Conn_01x02_Female -> Conn_01x03_Female; footprint Connector_PinHeader_2.54mm:PinHeader_1x02_P2.54mm_Vertical -> Connector_PinHeader_2.54mm:PinHeader_1x03_P2.54mm_Vertical; symbol Connector:Conn_01x02_Female -> Connector:Conn_01x03_Female
Connections:
- net RX: now also J.2 (Pin_2); no longer J.1 (Pin_1)
- net TX: now also J.3 (Pin_3); no longer J.2 (Pin_2)
- net RESET: now reaches Atmega1.1 (~{RESET}/PC6)
- net RESET: now also J.1 (Pin_1)
- no-connect marks 9 -> 8
Changed lines of the file:
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@@
   )
   (no_connect (at 196.85 344.17))
-  (no_connect (at 425.45 92.71))
   (no_connect (at 196.85 341.63))
   (no_connect (at 196.85 361.95))
@@
     (stroke (width 0) (type default) (color 0 0 0 0))
   )
-  (wire (pts (xy 425.45 92.71) (xy 422.91 92.71))
-    (stroke (width 0) (type default) (color 0 0 0 0))
-  )
   (wire (pts (xy 248.92 260.35) (xy 255.27 260.35))
     (stroke (width 0) (type default) (color 0 0 0 0))
@@
     (stroke (width 0) (type default) (color 0 0 0 0))
   )
+  (wire (pts (xy 452.12 93.98) (xy 454.66 93.98))
+    (stroke (width 0) (type default) (color 0 0 0 0))
+  )
   (polyline (pts (xy 163.83 236.22) (xy 163.83 375.92))
     (stroke (width 0) (type default) (color 0 0 0 0))
@@
     (stroke (width 0) (type default) (color 0 0 0 0))
   )
+  (wire (pts (xy 425.45 92.71) (xy 422.91 92.71))
+    (stroke (width 0) (type default) (color 0 0 0 0))
+  )
   (wire (pts (xy 391.16 189.23) (xy 393.7 189.23))
     (stroke (width 0) (type default) (color 0 0 0 0))
@@
     )
   )
+  (global_label "RESET" (shape output) (at 452.12 93.98 180) (fields_autoplaced)
+    (effects (font (size 1.27 1.27)) (justify right))
+    (property "Referenzen zwischen Schaltplänen" "${INTERSHEET_REFS}" (id 0) (at 443.9617 93.9006 0)
+      (effects (font (size 1.27 1.27)) (justify right) hide)
+    )
+  )
   (global_label "Row3" (shape input) (at 73.66 298.45 180) (fields_autoplaced)
     (effects (font (size 1.27 1.27)) (justify right))
@@
     )
   )
+  (global_label "RESET" (shape output) (at 425.45 92.71 0) (fields_autoplaced)
+    (effects (font (size 1.27 1.27)) (justify left))
+    (property "Referenzen zwischen Schaltplänen" "${INTERSHEET_REFS}" (id 0) (at 433.6083 92.6306 0)
+      (effects (font (size 1.27 1.27)) (justify left) hide)
+    )
+  )
   (global_label "trg2ToAtmega-b" (shape input) (at 425.45 105.41 0) (fields_autoplaced)
     (effects (font (size 1.27 1.27)) (justify left))
@@
     (pin "2")
   )
-  (symbol (lib_id "Connector:Conn_01x02_Female") (at 459.74 96.52 0) (unit 1)
+  (symbol (lib_id "Connector:Conn_01x03_Female") (at 459.74 96.52 0) (unit 1)
     (in_bom yes) (on_board yes) (fields_autoplaced)
-    (property "Reference" "J7" (id 0) (at 461.01 96.5199 0)
-      (effects (font (size 1.27 1.27)) (justify left))
-    )
-    (property "Value" "Conn_01x02_Female" (id 1) (at 461.01 99.0599 0)
-      (effects (font (size 1.27 1.27)) (justify left))
-    )
-    (property "Footprint" "Connector_PinHeader_2.54mm:PinHeader_1x02_P2.54mm_Vertical" (id 2) (at 459.74 96.52 0)
+    (property "Reference" "J7" (id 0) (at 459.74 91.44 0))
+    (property "Value" "Conn_01x03_Female" (id 1) (at 459.74 101.6 0))
+    (property "Footprint" "Connector_PinHeader_2.54mm:PinHeader_1x03_P2.54mm_Vertical" (id 2) (at 459.74 96.52 0)
       (effects (font (size 1.27 1.27)) hide)
     )
@@
       (effects (font (size 1.27 1.27)) hide)
     )
-    (property "Reference" "J?" (id 5) (at 459.74 96.52 0)
-      (effects (font (size 1.27 1.27)) hide)
-    )
-    (property "Value" "Conn_01x02_Female" (id 6) (at 459.74 96.52 0)
-      (effects (font (size 1.27 1.27)) hide)
-    )
+    (property "Reference" "J" (id 5) (at 459.74 91.44 0))
+    (property "Value" "Conn_01x03_Female" (id 6) (at 459.74 101.6 0))
     (pin "1")
     (pin "2")
+    (pin "3")
   )
   (symbol (lib_id "power:Earth") (at 139.7 34.29 0) (unit 1)
@@
     )
     (path "/8466e8ee-285b-4d22-85cb-418892ae7734"
-      (reference "J7") (unit 1) (value "Conn_01x02_Female") (footprint "Connector_PinHeader_2.54mm:PinHeader_1x02_P2.54mm_Vertical")
+      (reference "J7") (unit 1) (value "Conn_01x03_Female") (footprint "Connector_PinHeader_2.54mm:PinHeader_1x03_P2.54mm_Vertical")
     )
     (path "/5c9d9677-b457-410a-bc69-748e427b7183"
